Commit message: small changes to robot.xacro, new controller file robot.gazebo

File: warehouse_gz/models/simple_bot/robot.xacro (robot description, xacro)
@@ -45,5 +45,6 @@
 <xacro:macro name="inertia_body">
     <inertial>
-    <!-- displacement and orientation of the center of mass frame of the link with respect to the  -->
+    <!-- displacement and orientation of the center of mass frame of the link with respect to the coordinate plane -->
+    <!-- rpy stands for roll pitch yaw in the coordinate plane -->
     <origin rpy="0 0 0" xyz="0 0 ${s1}"/>
     <mass value"${m1}"/>
@@ -54,4 +55,5 @@
 <xacro:macro name="inertia_wheel">
     <inertial>
+    <!-- rotation around the x axis for the wheels represented in radians (its pi/2) -->
     <origin rpy="1.570795 0 0" xyz="0 0 0"/>
     <mass value="${m2}"/>
@@ -68,7 +70,8 @@
 </xacro:macro>
 <!-- ############################################################### -->
-<!-- Addidional files (may not be needed) -->
+<!-- Addidional files (needed for control) -->
 <!-- ############################################################### -->
-<!-- <xacro:include filename="$(find mobile_robot)/model/robot.gazebo"/> -->
+<!-- inside of the warehouse_gz package, in the models/simple_bot directory thats our file -->
+<xacro:include filename="$(find warehouse_gz)/models/simple_bot/robot.gazebo"/>
 <!-- ############################################################### -->
 <!-- Links and joints defenitions -->
@@ -84,11 +87,12 @@
     <visual>
         <geometry>
-            <box size="${a} ${b} ${c}"/>
+            <box size="${a} ${c} ${b}"/>
         </geometry>
+    <!-- displacement and orientation of the geometric center of the link with respect to the parent link-->
     <origin rpy="0 0 0" xyz="0 0 ${s1}"/>
     </visual>
     <collision>
         <geometry>
-            <box size="${a} ${b} ${c}"/>
+            <box size="${a} ${c} ${b}"/>
         </geometry>
     <origin rpy="0 0 0" xyz="0 0 ${s1}"/>

Commit message: simple robot up and running with teleop command, next step send commands thru commander node (HVBTA)

File: warehouse_gz/models/simple_bot/robot.xacro (robot description, xacro)
@@ -38,5 +38,5 @@
 <xacro:property name="Iz_body" value="${(1/12)*m1*(a*a+c*c)}"/>
 <!-- moments of inertia for the wheel -->
-<xacro:property name="Iz+wheel" value="${0.5*m2*r*r}"/>
+<xacro:property name="Iz_wheel" value="${0.5*m2*r*r}"/>
 <xacro:property name="I_wheel" value="${(1.0/12.0)*m2*(3.0*r*r+d*d)}"/>
 <!-- moments of inertia for the caster sphere -->
@@ -48,5 +48,5 @@
     <!-- rpy stands for roll pitch yaw in the coordinate plane -->
     <origin rpy="0 0 0" xyz="0 0 ${s1}"/>
-    <mass value"${m1}"/>
+    <mass value="${m1}"/>
     <inertia ixx="${Ix_body}" ixy="0.0" ixz="0.0" iyy="${Iy_body}" iyz="0.0" izz="${Iz_body}"/>
     </inertial>
@@ -58,5 +58,5 @@
     <origin rpy="1.570795 0 0" xyz="0 0 0"/>
     <mass value="${m2}"/>
-    <inertia ixx="${I_wheel}" ixy="0.0" ixz="0.0" iyy="${I_wheel}" iyz="0.0" izz="${Iz+wheel}"/>
+    <inertia ixx="${I_wheel}" ixy="0.0" ixz="0.0" iyy="${I_wheel}" iyz="0.0" izz="${Iz_wheel}"/>
     </inertial>
 </xacro:macro>

Commit message: added namespace to deal with multiple robots, each bot has its own bridge and state publisher now, added a clock bridge

File: warehouse_gz/models/simple_bot/robot.xacro (robot description, xacro)
@@ -16,4 +16,9 @@
 <xacro:property name="s3" value="${2*r}"/>
 <xacro:property name="s4" value="${c/2+d/2}"/>
+<!-- ############################################################### -->
+<!-- Define a robot namespace for multiple robots -->
+<!-- ############################################################### -->
+<xacro:arg name="robot_name" default="simple_bot"/>
+<xacro:property name="namespace" value="$(arg robot_name)"/>
 <!-- ############################################################ -->
 <!-- Mass and inertia -->
